Commit message: save

File: ros_gazebo/urdf/materials.xacro (robot description, xacro)
@@ -14,8 +14,8 @@
   </material>
   <material name="orange">
-    <color rgba="1.0 0.423529411765 0.0392156862745 1.0"/>
+    <color rgba="1.0 0.5 0.31 1.0"/>
   </material>
   <material name="brown">
-    <color rgba="0.870588235294 0.811764705882 0.764705882353 1.0"/>
+    <color rgba="0.55 0.27 0.075 1.0"/>
   </material>
   <material name="red">

File: ros_gazebo/urdf/robot.xacro (robot description, xacro)
@@ -7,9 +7,9 @@
   <xacro:include filename="$(find ros_gazebo)/urdf/robot.gazebo" />
   <xacro:include filename="$(find ros_gazebo)/urdf/macros.xacro" />
-	<xacro:property name="robot_mass" value="3" />
+	<xacro:property name="robot_mass" value="4" />
 	<xacro:property name="robot_height" value="1.165" />
 	<xacro:property name="robot_width" value="0.664" />
   <xacro:property name="robot_depth" value="0.33" />
-	<xacro:property name="module_mass" value="1" />
+	<xacro:property name="module_mass" value="2" />
 	<xacro:property name="module_height" value="1.161" />
 	<xacro:property name="module_width" value="0.664" />
