Commit message: update urdf

File: ros_gazebo/urdf/macros.xacro (robot description, xacro)
@@ -26,5 +26,5 @@
         <origin rpy="0 0 0" xyz="${origin_xyz}"/>
         <child link="${child}"/>
-        <parent link="link_chassis"/>
+        <parent link="base_footprint"/>
         <axis rpy="0 0 0" xyz="0 1 0"/>
         <limit effort="10000" velocity="1000"/>

File: ros_gazebo/urdf/materials.xacro (robot description, xacro)
@@ -5,8 +5,8 @@
   </material>
   <material name="blue">
-    <color rgba="0.203125 0.23828125 0.28515625 1.0"/>
+    <color rgba="0.0 0.0 1.0 1.0"/>
   </material>
   <material name="green">
-    <color rgba="0.0 0.8 0.0 1.0"/>
+    <color rgba="0.0 1.0 0.0 1.0"/>
   </material>
   <material name="grey">
@@ -20,5 +20,5 @@
   </material>
   <material name="red">
-    <color rgba="0.80078125 0.12890625 0.1328125 1.0"/>
+    <color rgba="1.0 0.0 0.0 1.0"/>
   </material>
   <material name="white">

File: ros_gazebo/urdf/robot.xacro (robot description, xacro)
@@ -1,80 +1,99 @@
 <?xml version="1.0" ?>
-<robot name="robot" xmlns:xacro="http://www.ros.org/wiki/xacro">
+<robot name="SASs_AMR_250" xmlns:xacro="http://www.ros.org/wiki/xacro">
+  <!-- base_footprint: tam xe tai mat phang ground -->
+  <!-- base_link: tam xe tai mat phang tam quay -->
+  <!-- base_laser: tam xe tai mat phang di qua tam laser -->
   <xacro:include filename="$(find ros_gazebo)/urdf/materials.xacro" />
   <xacro:include filename="$(find ros_gazebo)/urdf/robot.gazebo" />
   <xacro:include filename="$(find ros_gazebo)/urdf/macros.xacro" />
-  <link name="link_chassis">
-    <!-- pose and inertial -->
-    <pose>0 0 0.1 0 0 0</pose>
-    <inertial>
-      <mass value="5"/>
-      <origin rpy="0 0 0" xyz="0 0 0.1"/>
-      <inertia ixx="0.0395416666667" ixy="0" ixz="0" iyy="0.106208333333" iyz="0" izz="0.106208333333"/>
-    </inertial>
-    <!-- body -->
+  <link name="base_footprint">
+    <!-- <pose>0 0 0.1 0 0 0</pose> -->
+  </link>
+  <link name="base_link">
+    <!-- <inertial>
+      <origin xyz="0 0 0" rpy="0 0 0"/>
+      <mass value="120"/>
+      <inertia ixx="10.9" ixy="0.0" ixz="0.0"
+               iyy="5.125" iyz="0.0"
+               izz="14.225" />
+    </inertial> -->
+    <visual>
+      <origin xyz="0 0 -0.1" rpy="0 0 0"/>
+      <geometry>
+        <mesh filename="package://ros_gazebo/meshes/AMR_250.stl" scale="0.001 0.001 0.001"/>
+      </geometry>
+      <material name="red"/>
+    </visual>
     <collision name="collision_chassis">
       <geometry>
-        <box size="0.5 0.3 0.07"/>
+        <mesh filename="package://ros_gazebo/meshes/AMR_250.stl" scale="0.001 0.001 0.001"/>
       </geometry>
     </collision>
-    <visual>
-      <origin rpy="0 0 0" xyz="0 0 0"/>
-      <geometry>
-        <box size="0.5 0.3 0.07"/>
-      </geometry>
-      <material name="blue"/>
-    </visual>
-    <!-- caster front -->
-    <collision name="caster_front_collision">
-      <origin rpy="0 0 0" xyz="0.35 0 -0.05"/>
-      <geometry>
-        <sphere radius="0.05"/>
-      </geometry>
-      <surface>
-        <friction>
-          <ode>
-            <mu>0</mu>
-            <mu2>0</mu2>
-            <slip1>1.0</slip1>
-            <slip2>1.0</slip2>
-          </ode>
-        </friction>
-      </surface>
-    </collision>
-    <visual name="caster_front_visual">
-      <origin rpy=" 0 0 0" xyz="0.2 0 -0.05"/>
-      <geometry>
-        <sphere radius="0.05"/>
-      </geometry>
-    </visual>
   </link>
-  <link name="sensor_laser">
-    <inertial>
+  <joint name="base_link_joint" type="fixed">
+    <parent link="base_footprint"/>
+    <child link="base_link"/>
+    <origin xyz="0.0 0.0 0.1" rpy="0 0 0"/>
+  </joint>
+  <link name="base_laser">
+  </link>
+  <joint name="base_laser_joint" type="fixed">
+    <parent link="base_link"/>
+    <child link="base_laser"/>
+    <origin xyz="0 0 0.08" rpy="0 0 0"/>
+  </joint>
+  <link name="base_laser_front">
+    <!-- <inertial>
       <origin xyz="0 0 0" rpy="0 0 0" />
       <mass value="1" />
       <xacro:cylinder_inertia mass="1" r="0.05" l="0.1" />
-    </inertial>
+    </inertial> -->
     <visual>
-      <origin xyz="0 0 0" rpy="0 0 0" />
+      <origin xyz="0 0 0" rpy="0 0 0"/>
       <geometry>
-        <cylinder radius="0.05" length="0.1"/>
+        <mesh filename="package://ros_gazebo/meshes/ms3.stl" scale="0.01 0.01 0.01"/>
       </geometry>
-      <material name="white" />
+      <material name="blue"/>
     </visual>
     <collision>
       <origin xyz="0 0 0" rpy="0 0 0"/>
       <geometry>
-        <cylinder radius="0.05" length="0.1"/>
+        <mesh filename="package://ros_gazebo/meshes/ms3.stl" scale="0.01 0.01 0.01"/>
       </geometry>
     </collision>
   </link>
-  <joint name="joint_sensor_laser" type="fixed">
-    <origin xyz="0.15 0 0.05" rpy="0 0 0"/>
-    <parent link="link_chassis"/>
-    <child link="sensor_laser"/>
+  <joint name="base_laser_front_joint" type="fixed">
+    <parent link="base_laser"/>
+    <child link="base_laser_front"/>
+    <origin xyz="0.483 0.265 0" rpy="3.14 0 0.785"/>
   </joint>
-  <xacro:link_wheel name="link_right_wheel" />
-  <xacro:joint_wheel name="joint_right_wheel" child="link_right_wheel" origin_xyz="-0.05 0.20 0" />
-  <xacro:link_wheel name="link_left_wheel" />
-  <xacro:joint_wheel name="joint_left_wheel" child="link_left_wheel" origin_xyz="-0.05 -0.20 0" />
+  <link name="base_laser_back">
+    <!-- <inertial>
+      <origin xyz="0 0 0" rpy="0 0 0" />
+      <mass value="1" />
+      <xacro:cylinder_inertia mass="1" r="0.05" l="0.1" />
+    </inertial> -->
+    <visual>
+      <origin xyz="0 0 0" rpy="0 0 0"/>
+      <geometry>
+        <mesh filename="package://ros_gazebo/meshes/ms3.stl" scale="0.01 0.01 0.01"/>
+      </geometry>
+      <material name="blue"/>
+    </visual>
+    <collision>
+      <origin xyz="0 0 0" rpy="0 0 0"/>
+      <geometry>
+        <mesh filename="package://ros_gazebo/meshes/ms3.stl" scale="0.01 0.01 0.01"/>
+      </geometry>
+    </collision>
+  </link>
+  <joint name="base_laser_back_joint" type="fixed">
+    <parent link="base_laser"/>
+    <child link="base_laser_back"/>
+    <origin xyz="-0.483 -0.265 0" rpy="3.14 0 3.925"/>
+  </joint>
+  <xacro:link_wheel name="right_wheel" />
+  <xacro:joint_wheel name="joint_right_wheel" child="right_wheel" origin_xyz="0 0.20 0" />
+  <xacro:link_wheel name="left_wheel" />
+  <xacro:joint_wheel name="joint_left_wheel" child="left_wheel" origin_xyz="0 -0.20 0" />
 </robot>

Commit message: update urdf

File: ros_gazebo/urdf/macros.xacro (robot description, xacro)
@@ -11,5 +11,5 @@
               <origin rpy="0 1.5707 1.5707" xyz="0 0 0"/>
               <geometry>
-                <cylinder length="0.04" radius="0.1"/>
+                <cylinder length="0.046" radius="0.1"/>
               </geometry>
             </collision>
@@ -17,6 +17,7 @@
               <origin rpy="0 1.5707 1.5707" xyz="0 0 0"/>
               <geometry>
-                <cylinder length="0.04" radius="0.1"/>
+                <cylinder length="0.046" radius="0.1"/>
               </geometry>
+              <material name="green"/>
             </visual>
         </link>

File: ros_gazebo/urdf/robot.xacro (robot description, xacro)
@@ -19,5 +19,5 @@
     </inertial> -->
     <visual>
-      <origin xyz="0 0 -0.1" rpy="0 0 0"/>
+      <origin xyz="0 0 -0.1" rpy="0 0 1.57"/>
       <geometry>
         <mesh filename="package://ros_gazebo/meshes/AMR_250.stl" scale="0.001 0.001 0.001"/>
@@ -94,6 +94,6 @@
   </joint>
   <xacro:link_wheel name="right_wheel" />
-  <xacro:joint_wheel name="joint_right_wheel" child="right_wheel" origin_xyz="0 0.20 0" />
+  <xacro:joint_wheel name="joint_right_wheel" child="right_wheel" origin_xyz="0 0.242 0.1" />
   <xacro:link_wheel name="left_wheel" />
-  <xacro:joint_wheel name="joint_left_wheel" child="left_wheel" origin_xyz="0 -0.20 0" />
+  <xacro:joint_wheel name="joint_left_wheel" child="left_wheel" origin_xyz="0 -0.242 0.1" />
 </robot>

Commit message: update world

File: ros_gazebo/urdf/macros.xacro (robot description, xacro)
@@ -38,3 +38,8 @@
                 izz="${mass*(r*r)/2}" />
     </xacro:macro>
+    <xacro:macro name="solid_cuboid_inertia" params="m h w d">
+      <inertia  ixx="${(m*(h*h+d*d))/12}" ixy = "0" ixz = "0"
+                iyy="${(m*(w*w+h*h))/12}" iyz = "0"
+                izz="${(m*(w*w+d*d))/12}" />
+    </xacro:macro>
 </robot>

File: ros_gazebo/urdf/robot.xacro (robot description, xacro)
@@ -7,4 +7,8 @@
   <xacro:include filename="$(find ros_gazebo)/urdf/robot.gazebo" />
   <xacro:include filename="$(find ros_gazebo)/urdf/macros.xacro" />
+	<xacro:property name="robot_mass" value="150" />
+	<xacro:property name="robot_height" value="1.161" />
+	<xacro:property name="robot_width" value="0.664" />
+  <xacro:property name="robot_depth" value="0.33" />
   <link name="base_footprint">
     <!-- <pose>0 0 0.1 0 0 0</pose> -->
@@ -13,11 +17,9 @@
     <!-- <inertial>
       <origin xyz="0 0 0" rpy="0 0 0"/>
-      <mass value="120"/>
-      <inertia ixx="10.9" ixy="0.0" ixz="0.0"
-               iyy="5.125" iyz="0.0"
-               izz="14.225" />
+      <mass value="${robot_mass}" />
+      <solid_cuboid_inertia m="${robot_mass}" h="${robot_height}" w="${robot_width}" d="${robot_depth}"/>
     </inertial> -->
     <visual>
-      <origin xyz="0 0 -0.1" rpy="0 0 1.57"/>
+      <origin xyz="0 0 -0.1" rpy="0 0 -1.57"/>
       <geometry>
         <mesh filename="package://ros_gazebo/meshes/AMR_250.stl" scale="0.001 0.001 0.001"/>
@@ -50,5 +52,5 @@
     </inertial> -->
     <visual>
-      <origin xyz="0 0 0" rpy="0 0 0"/>
+      <origin xyz="0 0 0" rpy="0 0 -2.355"/>
       <geometry>
         <mesh filename="package://ros_gazebo/meshes/ms3.stl" scale="0.01 0.01 0.01"/>
@@ -57,5 +59,5 @@
     </visual>
     <collision>
-      <origin xyz="0 0 0" rpy="0 0 0"/>
+      <origin xyz="0 0 0" rpy="0 0 -2.355"/>
       <geometry>
         <mesh filename="package://ros_gazebo/meshes/ms3.stl" scale="0.01 0.01 0.01"/>
@@ -75,5 +77,5 @@
     </inertial> -->
     <visual>
-      <origin xyz="0 0 0" rpy="0 0 0"/>
+      <origin xyz="0 0 0" rpy="0 0 -0.785"/>
       <geometry>
         <mesh filename="package://ros_gazebo/meshes/ms3.stl" scale="0.01 0.01 0.01"/>
@@ -82,5 +84,5 @@
     </visual>
     <collision>
-      <origin xyz="0 0 0" rpy="0 0 0"/>
+      <origin xyz="0 0 0" rpy="0 0 -0.785"/>
       <geometry>
         <mesh filename="package://ros_gazebo/meshes/ms3.stl" scale="0.01 0.01 0.01"/>

Commit message: save

File: ros_gazebo/urdf/macros.xacro (robot description, xacro)
@@ -8,5 +8,5 @@
               <inertia ixx="0.000526666666667" ixy="0" ixz="0" iyy="0.000526666666667" iyz="0" izz="0.001"/>
             </inertial>
-            <collision name="link_right_wheel_collision">
+            <collision name="${name}_collision">
               <origin rpy="0 1.5707 1.5707" xyz="0 0 0"/>
               <geometry>

Commit message: test good

File: ros_gazebo/urdf/macros.xacro (robot description, xacro)
@@ -27,5 +27,5 @@
         <origin rpy="0 0 0" xyz="${origin_xyz}"/>
         <child link="${child}"/>
-        <parent link="base_footprint"/>
+        <parent link="base_link"/>
         <axis rpy="0 0 0" xyz="0 1 0"/>
         <limit effort="10000" velocity="1000"/>

File: ros_gazebo/urdf/robot.xacro (robot description, xacro)
@@ -7,9 +7,9 @@
   <xacro:include filename="$(find ros_gazebo)/urdf/robot.gazebo" />
   <xacro:include filename="$(find ros_gazebo)/urdf/macros.xacro" />
-	<xacro:property name="robot_mass" value="200" />
-	<xacro:property name="robot_height" value="0.95" />
-	<xacro:property name="robot_width" value="0.48" />
+	<xacro:property name="robot_mass" value="5" />
+	<xacro:property name="robot_height" value="1.165" />
+	<xacro:property name="robot_width" value="0.664" />
   <xacro:property name="robot_depth" value="0.33" />
-	<xacro:property name="module_mass" value="40" />
+	<xacro:property name="module_mass" value="5" />
 	<xacro:property name="module_height" value="1.161" />
 	<xacro:property name="module_width" value="0.664" />
@@ -21,10 +21,10 @@
     <pose>0 0 0 0 0 0</pose>
     <inertial>
-      <origin xyz="0 0 -0.07" rpy="0 0 0"/>
+      <origin xyz="0 0 -0.069" rpy="0 0 0"/>
       <mass value="${robot_mass}" />
       <solid_cuboid_inertia m="${robot_mass}" h="${robot_height}" w="${robot_width}" d="${robot_depth}"/>
     </inertial>
     <visual>
-      <origin xyz="0 0 -0.07" rpy="0 0 0"/>
+      <origin xyz="0 0 -0.069" rpy="0 0 0"/>
       <geometry>
         <!-- <box size="${robot_width} ${robot_height} ${robot_depth}"/> -->
@@ -34,5 +34,5 @@
     </visual>
     <collision name="base_link">
-      <origin xyz="0 0 -0.07" rpy="0 0 0"/>
+      <origin xyz="0 0 -0.069" rpy="0 0 0"/>
       <geometry>
         <!-- <box size="${robot_width} ${robot_height} ${robot_depth}"/> -->
@@ -56,5 +56,5 @@
     <origin xyz="0.0 0.0 0.1" rpy="0 0 0"/>
   </joint>
-  <link name="base_module"></link>
+  <!-- <link name="base_module"></link>
   <joint name="base_module_joint" type="fixed">
     <parent link="base_link"/>
@@ -111,5 +111,5 @@
     <child link="base_module_up"/>
     <origin xyz="0.0 0.0 0.0" rpy="0 0 0"/>
-  </joint>
+  </joint> -->
   <link name="base_laser"></link>
   <joint name="base_laser_joint" type="fixed">
@@ -169,6 +169,6 @@
   </joint>
   <xacro:link_wheel name="right_wheel" />
-  <xacro:joint_wheel name="joint_right_wheel" child="right_wheel" origin_xyz="0 0.242 0.1" />
+  <xacro:joint_wheel name="joint_right_wheel" child="right_wheel" origin_xyz="0 0.242 0" />
   <xacro:link_wheel name="left_wheel" />
-  <xacro:joint_wheel name="joint_left_wheel" child="left_wheel" origin_xyz="0 -0.242 0.1" />
+  <xacro:joint_wheel name="joint_left_wheel" child="left_wheel" origin_xyz="0 -0.242 0" />
 </robot>

Commit message: save

File: ros_gazebo/urdf/macros.xacro (robot description, xacro)
@@ -1,45 +1,82 @@
 <?xml version="1.0"?>
 <robot xmlns:xacro="http://www.ros.org/wiki/xacro">
-    <xacro:macro name="link_wheel" params="name">
-        <link name="${name}">
-            <inertial>
-              <mass value="0.2"/>
-              <origin rpy="0 1.5707 1.5707" xyz="0 0 0"/>
-              <inertia ixx="0.000526666666667" ixy="0" ixz="0" iyy="0.000526666666667" iyz="0" izz="0.001"/>
-            </inertial>
-            <collision name="${name}_collision">
-              <origin rpy="0 1.5707 1.5707" xyz="0 0 0"/>
-              <geometry>
-                <cylinder length="0.046" radius="0.1"/>
-              </geometry>
-            </collision>
-            <visual name="${name}_visual">
-              <origin rpy="0 1.5707 1.5707" xyz="0 0 0"/>
-              <geometry>
-                <cylinder length="0.046" radius="0.1"/>
-              </geometry>
-              <material name="green"/>
-            </visual>
-        </link>
-    </xacro:macro>
-    <xacro:macro name="joint_wheel" params="name child origin_xyz">
-      <joint name="${name}" type="continuous">
-        <origin rpy="0 0 0" xyz="${origin_xyz}"/>
-        <child link="${child}"/>
-        <parent link="base_link"/>
-        <axis rpy="0 0 0" xyz="0 1 0"/>
-        <limit effort="10000" velocity="1000"/>
-        <joint_properties damping="1.0" friction="1.0"/>
-      </joint>
-    </xacro:macro>
-    <xacro:macro name="cylinder_inertia" params="mass r l">
-      <inertia  ixx="${mass*(3*r*r+l*l)/12}" ixy = "0" ixz = "0"
-                iyy="${mass*(3*r*r+l*l)/12}" iyz = "0"
-                izz="${mass*(r*r)/2}" />
-    </xacro:macro>
-    <xacro:macro name="solid_cuboid_inertia" params="m h w d">
-      <inertia  ixx="${(m*(h*h+d*d))/12}" ixy = "0" ixz = "0"
-                iyy="${(m*(w*w+h*h))/12}" iyz = "0"
-                izz="${(m*(w*w+d*d))/12}" />
-    </xacro:macro>
+  <xacro:macro name="link_wheel" params="name">
+      <link name="${name}">
+          <inertial>
+            <mass value="0.2"/>
+            <origin rpy="0 1.5707 1.5707" xyz="0 0 0"/>
+            <inertia ixx="0.000526666666667" ixy="0" ixz="0" iyy="0.000526666666667" iyz="0" izz="0.001"/>
+          </inertial>
+          <collision name="${name}_collision">
+            <origin rpy="0 1.5707 1.5707" xyz="0 0 0"/>
+            <geometry>
+              <cylinder length="0.046" radius="0.1"/>
+            </geometry>
+          </collision>
+          <visual name="${name}_visual">
+            <origin rpy="0 1.5707 1.5707" xyz="0 0 0"/>
+            <geometry>
+              <cylinder length="0.046" radius="0.1"/>
+            </geometry>
+            <material name="green"/>
+          </visual>
+      </link>
+  </xacro:macro>
+  <xacro:macro name="joint_wheel" params="name parent child origin_xyz">
+    <joint name="${name}" type="continuous">
+      <origin rpy="0 0 0" xyz="${origin_xyz}"/>
+      <child link="${child}"/>
+      <parent link="${parent}"/>
+      <axis rpy="0 0 0" xyz="0 1 0"/>
+      <limit effort="10000" velocity="1000"/>
+      <joint_properties damping="1.0" friction="1.0"/>
+    </joint>
+  </xacro:macro>
+  <xacro:macro name="joint_module" params="name parent child origin_xyz">
+    <joint name="${name}" type="fixed">
+      <!-- <joint_properties damping="1.0" friction="1.0"/> -->
+      <child link="${child}"/>
+      <parent link="${parent}"/>
+      <!-- <pose frame=''>0 0 0 0 0 0</pose> -->
+      <origin rpy="0 0 0" xyz="${origin_xyz}"/>
+      <axis>
+        <xyz>0 0 1</xyz>
+        <use_parent_model_frame>0</use_parent_model_frame>
+        <limit>
+          <lower>0</lower>
+          <upper>0.25</upper>
+          <effort>-1</effort>
+          <velocity>-1</velocity>
+        </limit>
+        <dynamics>
+          <spring_reference>0</spring_reference>
+          <spring_stiffness>0</spring_stiffness>
+          <damping>0</damping>
+          <friction>0</friction>
+        </dynamics>
+      </axis>
+      <physics>
+        <ode>
+          <limit>
+            <cfm>0</cfm>
+            <erp>0.2</erp>
+          </limit>
+          <suspension>
+            <cfm>0</cfm>
+            <erp>0.2</erp>
+          </suspension>
+        </ode>
+      </physics>
+    </joint>
+  </xacro:macro>
+  <xacro:macro name="cylinder_inertia" params="mass r l">
+    <inertia  ixx="${mass*(3*r*r+l*l)/12}" ixy = "0" ixz = "0"
+              iyy="${mass*(3*r*r+l*l)/12}" iyz = "0"
+              izz="${mass*(r*r)/2}" />
+  </xacro:macro>
+  <xacro:macro name="solid_cuboid_inertia" params="m h w d">
+    <inertia  ixx="${(m*(h*h+d*d))/12}" ixy = "0" ixz = "0"
+              iyy="${(m*(w*w+h*h))/12}" iyz = "0"
+              izz="${(m*(w*w+d*d))/12}" />
+  </xacro:macro>
 </robot>

File: ros_gazebo/urdf/robot.xacro (robot description, xacro)
@@ -51,5 +51,5 @@
     <origin xyz="0.0 0.0 0.1" rpy="0 0 0"/>
   </joint>
-  <!-- <link name="base_module"></link>
+  <link name="base_module"></link>
   <joint name="base_module_joint" type="fixed">
     <parent link="base_link"/>
@@ -57,5 +57,5 @@
     <origin xyz="0 0 0.23" rpy="0 0 -1.57"/>
   </joint>
-  <link name="base_module_under">
+  <link name="module_under">
     <inertial>
       <origin xyz="0 0 0" rpy="0 0 0" />
@@ -79,8 +79,8 @@
   <joint name="base_module_under_joint" type="fixed">
     <parent link="base_module"/>
-    <child link="base_module_under"/>
+    <child link="module_under"/>
     <origin xyz="0.0 0.0 0.0" rpy="0 0 0"/>
   </joint>
-  <link name="base_module_up">
+  <link name="module_up">
     <inertial>
       <origin xyz="0 0 0" rpy="0 0 0" />
@@ -102,10 +102,6 @@
     </collision>
   </link>
-  <joint name="base_module_up_joint" type="fixed">
-    <parent link="base_module"/>
-    <child link="base_module_up"/>
-    <origin xyz="0.0 0.0 0.0" rpy="0 0 0"/>
-  </joint> -->
-  <!-- <link name="base_laser"></link>
+  <xacro:joint_module name="lift" parent="base_module" child="module_up" origin_xyz="0 0 0" />
+  <link name="base_laser"></link>
   <joint name="base_laser_joint" type="fixed">
     <parent link="base_link"/>
@@ -187,8 +183,8 @@
     <child link="base_camera"/>
     <origin xyz="0.53 0 0.15" rpy="0 0 0"/>
-  </joint> -->
+  </joint>
   <xacro:link_wheel name="right_wheel" />
-  <xacro:joint_wheel name="joint_right_wheel" child="right_wheel" origin_xyz="0 -0.242 0" />
+  <xacro:joint_wheel name="joint_right_wheel" parent="base_link" child="right_wheel" origin_xyz="0 -0.242 0" />
   <xacro:link_wheel name="left_wheel" />
-  <xacro:joint_wheel name="joint_left_wheel" child="left_wheel" origin_xyz="0 0.242 0" />
+  <xacro:joint_wheel name="joint_left_wheel" parent="base_link" child="left_wheel" origin_xyz="0 0.242 0" />
 </robot>

Commit message: save

File: ros_gazebo/urdf/macros.xacro (robot description, xacro)
@@ -34,26 +34,11 @@
   </xacro:macro>
   <xacro:macro name="joint_module" params="name parent child origin_xyz">
-    <joint name="${name}" type="fixed">
-      <!-- <joint_properties damping="1.0" friction="1.0"/> -->
+    <joint name="${name}" type="prismatic">
       <child link="${child}"/>
       <parent link="${parent}"/>
-      <!-- <pose frame=''>0 0 0 0 0 0</pose> -->
       <origin rpy="0 0 0" xyz="${origin_xyz}"/>
-      <axis>
-        <xyz>0 0 1</xyz>
-        <use_parent_model_frame>0</use_parent_model_frame>
-        <limit>
-          <lower>0</lower>
-          <upper>0.25</upper>
-          <effort>-1</effort>
-          <velocity>-1</velocity>
-        </limit>
-        <dynamics>
-          <spring_reference>0</spring_reference>
-          <spring_stiffness>0</spring_stiffness>
-          <damping>0</damping>
-          <friction>0</friction>
-        </dynamics>
-      </axis>
+      <axis xyz="0 0 1"/>
+	    <limit lower="0.0" upper="0.25" effort="1000" velocity="1"/>
+	    <dynamics spring_reference="0" spring_stiffness="0" damping="1" friction="1"/>
       <physics>
         <ode>

Commit message: save

File: ros_gazebo/urdf/macros.xacro (robot description, xacro)
@@ -39,6 +39,6 @@
       <origin rpy="0 0 0" xyz="${origin_xyz}"/>
       <axis xyz="0 0 1"/>
-	    <limit lower="0.0" upper="0.25" effort="1000" velocity="1"/>
-	    <dynamics spring_reference="0" spring_stiffness="0" damping="1" friction="1"/>
+	    <limit lower="0.0" upper="0.05" effort="1000" velocity="1"/>
+	    <dynamics spring_reference="0" spring_stiffness="0" damping="0" friction="0"/>
       <physics>
         <ode>

Commit message: save

File: ros_gazebo/urdf/macros.xacro (robot description, xacro)
@@ -39,6 +39,6 @@
       <origin rpy="0 0 0" xyz="${origin_xyz}"/>
       <axis xyz="0 0 1"/>
-	    <limit lower="0.0" upper="0.05" effort="1000" velocity="1"/>
-	    <dynamics spring_reference="0" spring_stiffness="0" damping="0" friction="0"/>
+	    <limit lower="0.0" upper="0.05" effort="10000" velocity="0.5"/>
+	    <dynamics spring_reference="0.8" spring_stiffness="50" damping="1" friction="10"/>
       <physics>
         <ode>
