Commit message: add AMR_250

File: ros_gazebo/urdf/robot.xacro (robot description, xacro)
@@ -27,5 +27,5 @@
     <!-- caster front -->
     <collision name="caster_front_collision">
-      <origin rpy=" 0 0 0" xyz="0.35 0 -0.05"/>
+      <origin rpy="0 0 0" xyz="0.35 0 -0.05"/>
       <geometry>
         <sphere radius="0.05"/>

Commit message: update

File: ros_gazebo/urdf/robot.xacro (robot description, xacro)
@@ -52,14 +52,14 @@
     </inertial> -->
     <visual>
-      <origin xyz="0 0 0" rpy="0 0 -2.355"/>
+      <origin xyz="0 0 0" rpy="0 0 3.14"/>
       <geometry>
-        <mesh filename="package://ros_gazebo/meshes/ms3.stl" scale="0.01 0.01 0.01"/>
+        <mesh filename="package://ros_gazebo/meshes/ms3.stl" scale="0.001 0.001 0.001"/>
       </geometry>
       <material name="blue"/>
     </visual>
     <collision>
-      <origin xyz="0 0 0" rpy="0 0 -2.355"/>
+      <origin xyz="0 0 0" rpy="0 0 3.14"/>
       <geometry>
-        <mesh filename="package://ros_gazebo/meshes/ms3.stl" scale="0.01 0.01 0.01"/>
+        <mesh filename="package://ros_gazebo/meshes/ms3.stl" scale="0.001 0.001 0.001"/>
       </geometry>
     </collision>
@@ -77,14 +77,14 @@
     </inertial> -->
     <visual>
-      <origin xyz="0 0 0" rpy="0 0 -0.785"/>
+      <origin xyz="0 0 0" rpy="0 0 3.14"/>
       <geometry>
-        <mesh filename="package://ros_gazebo/meshes/ms3.stl" scale="0.01 0.01 0.01"/>
+        <mesh filename="package://ros_gazebo/meshes/ms3.stl" scale="0.001 0.001 0.001"/>
       </geometry>
       <material name="blue"/>
     </visual>
     <collision>
-      <origin xyz="0 0 0" rpy="0 0 -0.785"/>
+      <origin xyz="0 0 0" rpy="0 0 3.14"/>
       <geometry>
-        <mesh filename="package://ros_gazebo/meshes/ms3.stl" scale="0.01 0.01 0.01"/>
+        <mesh filename="package://ros_gazebo/meshes/ms3.stl" scale="0.001 0.001 0.001"/>
       </geometry>
     </collision>

Commit message: update

File: ros_gazebo/urdf/robot.xacro (robot description, xacro)
@@ -52,5 +52,5 @@
     </inertial> -->
     <visual>
-      <origin xyz="0 0 0" rpy="0 0 3.14"/>
+      <origin xyz="0 0 0" rpy="0 0 0"/>
       <geometry>
         <mesh filename="package://ros_gazebo/meshes/ms3.stl" scale="0.001 0.001 0.001"/>
@@ -59,5 +59,5 @@
     </visual>
     <collision>
-      <origin xyz="0 0 0" rpy="0 0 3.14"/>
+      <origin xyz="0 0 0" rpy="0 0 0"/>
       <geometry>
         <mesh filename="package://ros_gazebo/meshes/ms3.stl" scale="0.001 0.001 0.001"/>
@@ -77,5 +77,5 @@
     </inertial> -->
     <visual>
-      <origin xyz="0 0 0" rpy="0 0 3.14"/>
+      <origin xyz="0 0 0" rpy="0 0 0"/>
       <geometry>
         <mesh filename="package://ros_gazebo/meshes/ms3.stl" scale="0.001 0.001 0.001"/>
@@ -84,5 +84,5 @@
     </visual>
     <collision>
-      <origin xyz="0 0 0" rpy="0 0 3.14"/>
+      <origin xyz="0 0 0" rpy="0 0 0"/>
       <geometry>
         <mesh filename="package://ros_gazebo/meshes/ms3.stl" scale="0.001 0.001 0.001"/>

Commit message: add module

File: ros_gazebo/urdf/robot.xacro (robot description, xacro)
@@ -38,6 +38,61 @@
     <origin xyz="0.0 0.0 0.1" rpy="0 0 0"/>
   </joint>
-  <link name="base_laser">
+  <link name="base_module"></link>
+  <joint name="base_module_joint" type="fixed">
+    <parent link="base_link"/>
+    <child link="base_module"/>
+    <origin xyz="0 0 0.23" rpy="0 0 -1.57"/>
+  </joint>
+  <link name="base_module_under">
+    <!-- <inertial>
+      <origin xyz="0 0 0" rpy="0 0 0" />
+      <mass value="1" />
+      <xacro:cylinder_inertia mass="1" r="0.05" l="0.1" />
+    </inertial> -->
+    <visual>
+      <origin xyz="0 0 0" rpy="0 0 0"/>
+      <geometry>
+        <mesh filename="package://ros_gazebo/meshes/AMR_Module1.stl" scale="0.001 0.001 0.001"/>
+      </geometry>
+      <material name="orange"/>
+    </visual>
+    <collision>
+      <origin xyz="0 0 0" rpy="0 0 0"/>
+      <geometry>
+        <mesh filename="package://ros_gazebo/meshes/AMR_Module1.stl" scale="0.001 0.001 0.001"/>
+      </geometry>
+    </collision>
   </link>
+  <joint name="base_module_under_joint" type="fixed">
+    <parent link="base_module"/>
+    <child link="base_module_under"/>
+    <origin xyz="0.0 0.0 0.0" rpy="0 0 0"/>
+  </joint>
+  <link name="base_module_up">
+    <!-- <inertial>
+      <origin xyz="0 0 0" rpy="0 0 0" />
+      <mass value="1" />
+      <xacro:cylinder_inertia mass="1" r="0.05" l="0.1" />
+    </inertial> -->
+    <visual>
+      <origin xyz="0 0 0" rpy="0 0 0"/>
+      <geometry>
+        <mesh filename="package://ros_gazebo/meshes/AMR_Module2.stl" scale="0.001 0.001 0.001"/>
+      </geometry>
+      <material name="brown"/>
+    </visual>
+    <collision>
+      <origin xyz="0 0 0" rpy="0 0 0"/>
+      <geometry>
+        <mesh filename="package://ros_gazebo/meshes/AMR_Module2.stl" scale="0.001 0.001 0.001"/>
+      </geometry>
+    </collision>
+  </link>
+  <joint name="base_module_up_joint" type="fixed">
+    <parent link="base_module"/>
+    <child link="base_module_up"/>
+    <origin xyz="0.0 0.0 0.0" rpy="0 0 0"/>
+  </joint>
+  <link name="base_laser"></link>
   <joint name="base_laser_joint" type="fixed">
     <parent link="base_link"/>

Commit message: save

File: ros_gazebo/urdf/robot.xacro (robot description, xacro)
@@ -10,17 +10,22 @@
 	<xacro:property name="robot_height" value="1.161" />
 	<xacro:property name="robot_width" value="0.664" />
-  <xacro:property name="robot_depth" value="0.33" />
+  <xacro:property name="robot_depth" value="0.3" />
+	<xacro:property name="module_mass" value="40" />
+	<xacro:property name="module_height" value="1.161" />
+	<xacro:property name="module_width" value="0.664" />
+  <xacro:property name="module_depth" value="0.15" />
   <link name="base_footprint">
     <!-- <pose>0 0 0.1 0 0 0</pose> -->
   </link>
   <link name="base_link">
-    <!-- <inertial>
+    <inertial>
       <origin xyz="0 0 0" rpy="0 0 0"/>
       <mass value="${robot_mass}" />
       <solid_cuboid_inertia m="${robot_mass}" h="${robot_height}" w="${robot_width}" d="${robot_depth}"/>
-    </inertial> -->
+    </inertial>
     <visual>
       <origin xyz="0 0 -0.1" rpy="0 0 -1.57"/>
       <geometry>
+        <!-- <box size="1 1 0.3" /> -->
         <mesh filename="package://ros_gazebo/meshes/AMR_250.stl" scale="0.001 0.001 0.001"/>
       </geometry>
@@ -29,4 +34,5 @@
     <collision name="collision_chassis">
       <geometry>
+        <!-- <box size="1 1 0.3" /> -->
         <mesh filename="package://ros_gazebo/meshes/AMR_250.stl" scale="0.001 0.001 0.001"/>
       </geometry>
@@ -45,9 +51,9 @@
   </joint>
   <link name="base_module_under">
-    <!-- <inertial>
+    <inertial>
       <origin xyz="0 0 0" rpy="0 0 0" />
-      <mass value="1" />
-      <xacro:cylinder_inertia mass="1" r="0.05" l="0.1" />
-    </inertial> -->
+      <mass value="${module_mass}" />
+      <solid_cuboid_inertia m="${module_mass}" h="${module_height}" w="${module_width}" d="${module_depth}"/>
+    </inertial>
     <visual>
       <origin xyz="0 0 0" rpy="0 0 0"/>
@@ -70,9 +76,9 @@
   </joint>
   <link name="base_module_up">
-    <!-- <inertial>
+    <inertial>
       <origin xyz="0 0 0" rpy="0 0 0" />
-      <mass value="1" />
-      <xacro:cylinder_inertia mass="1" r="0.05" l="0.1" />
-    </inertial> -->
+      <mass value="${module_mass}" />
+      <solid_cuboid_inertia m="${module_mass}" h="${module_height}" w="${module_width}" d="${module_depth}"/>
+    </inertial>
     <visual>
       <origin xyz="0 0 0" rpy="0 0 0"/>
@@ -101,9 +107,9 @@
   </joint>
   <link name="base_laser_front">
-    <!-- <inertial>
+    <inertial>
       <origin xyz="0 0 0" rpy="0 0 0" />
       <mass value="1" />
       <xacro:cylinder_inertia mass="1" r="0.05" l="0.1" />
-    </inertial> -->
+    </inertial>
     <visual>
       <origin xyz="0 0 0" rpy="0 0 0"/>
@@ -126,9 +132,9 @@
   </joint>
   <link name="base_laser_back">
-    <!-- <inertial>
+    <inertial>
       <origin xyz="0 0 0" rpy="0 0 0" />
       <mass value="1" />
       <xacro:cylinder_inertia mass="1" r="0.05" l="0.1" />
-    </inertial> -->
+    </inertial>
     <visual>
       <origin xyz="0 0 0" rpy="0 0 0"/>

Commit message: save

File: ros_gazebo/urdf/robot.xacro (robot description, xacro)
@@ -7,8 +7,8 @@
   <xacro:include filename="$(find ros_gazebo)/urdf/robot.gazebo" />
   <xacro:include filename="$(find ros_gazebo)/urdf/macros.xacro" />
-	<xacro:property name="robot_mass" value="150" />
+	<xacro:property name="robot_mass" value="200" />
 	<xacro:property name="robot_height" value="1.161" />
 	<xacro:property name="robot_width" value="0.664" />
-  <xacro:property name="robot_depth" value="0.3" />
+  <xacro:property name="robot_depth" value="0.33" />
 	<xacro:property name="module_mass" value="40" />
 	<xacro:property name="module_height" value="1.161" />
@@ -20,20 +20,21 @@
   <link name="base_link">
     <inertial>
-      <origin xyz="0 0 0" rpy="0 0 0"/>
+    <origin xyz="0 0 0.1" rpy="0 0 -1.57"/>
       <mass value="${robot_mass}" />
       <solid_cuboid_inertia m="${robot_mass}" h="${robot_height}" w="${robot_width}" d="${robot_depth}"/>
     </inertial>
     <visual>
-      <origin xyz="0 0 -0.1" rpy="0 0 -1.57"/>
+      <origin xyz="0 0 0.1" rpy="0 0 -1.57"/>
       <geometry>
-        <!-- <box size="1 1 0.3" /> -->
-        <mesh filename="package://ros_gazebo/meshes/AMR_250.stl" scale="0.001 0.001 0.001"/>
+        <box size="${robot_width} ${robot_height} ${robot_depth}"/>
+        <!-- <mesh filename="package://ros_gazebo/meshes/AMR_250.stl" scale="0.001 0.001 0.001"/> -->
       </geometry>
       <material name="red"/>
     </visual>
-    <collision name="collision_chassis">
+    <collision name="base_link">
+      <origin xyz="0 0 0.1" rpy="0 0 -1.57"/>
       <geometry>
-        <!-- <box size="1 1 0.3" /> -->
-        <mesh filename="package://ros_gazebo/meshes/AMR_250.stl" scale="0.001 0.001 0.001"/>
+        <box size="${robot_width} ${robot_height} ${robot_depth}"/>
+        <!-- <mesh filename="package://ros_gazebo/meshes/AMR_250.stl" scale="0.001 0.001 0.001"/> -->
       </geometry>
     </collision>

Commit message: save

File: ros_gazebo/urdf/robot.xacro (robot description, xacro)
@@ -8,6 +8,6 @@
   <xacro:include filename="$(find ros_gazebo)/urdf/macros.xacro" />
 	<xacro:property name="robot_mass" value="200" />
-	<xacro:property name="robot_height" value="1.161" />
-	<xacro:property name="robot_width" value="0.664" />
+	<xacro:property name="robot_height" value="0.95" />
+	<xacro:property name="robot_width" value="0.5" />
   <xacro:property name="robot_depth" value="0.33" />
 	<xacro:property name="module_mass" value="40" />

Commit message: save

File: ros_gazebo/urdf/robot.xacro (robot description, xacro)
@@ -9,5 +9,5 @@
 	<xacro:property name="robot_mass" value="200" />
 	<xacro:property name="robot_height" value="0.95" />
-	<xacro:property name="robot_width" value="0.5" />
+	<xacro:property name="robot_width" value="0.48" />
   <xacro:property name="robot_depth" value="0.33" />
 	<xacro:property name="module_mass" value="40" />
@@ -16,5 +16,4 @@
   <xacro:property name="module_depth" value="0.15" />
   <link name="base_footprint">
-    <!-- <pose>0 0 0.1 0 0 0</pose> -->
   </link>
   <link name="base_link">

Commit message: save

File: ros_gazebo/urdf/robot.xacro (robot description, xacro)
@@ -16,25 +16,37 @@
   <xacro:property name="module_depth" value="0.15" />
   <link name="base_footprint">
+    <origin xyz="0 0 0" rpy="0 0 -1.57"/>
   </link>
   <link name="base_link">
+    <pose>0 0 0 0 0 0</pose>
     <inertial>
-    <origin xyz="0 0 0.1" rpy="0 0 -1.57"/>
+      <origin xyz="0 0 -0.07" rpy="0 0 0"/>
       <mass value="${robot_mass}" />
       <solid_cuboid_inertia m="${robot_mass}" h="${robot_height}" w="${robot_width}" d="${robot_depth}"/>
     </inertial>
     <visual>
-      <origin xyz="0 0 0.1" rpy="0 0 -1.57"/>
+      <origin xyz="0 0 -0.07" rpy="0 0 0"/>
       <geometry>
-        <box size="${robot_width} ${robot_height} ${robot_depth}"/>
-        <!-- <mesh filename="package://ros_gazebo/meshes/AMR_250.stl" scale="0.001 0.001 0.001"/> -->
+        <!-- <box size="${robot_width} ${robot_height} ${robot_depth}"/> -->
+        <mesh filename="package://ros_gazebo/meshes/AMR_250.stl" scale="0.001 0.001 0.001"/>
       </geometry>
       <material name="red"/>
     </visual>
     <collision name="base_link">
-      <origin xyz="0 0 0.1" rpy="0 0 -1.57"/>
+      <origin xyz="0 0 -0.07" rpy="0 0 0"/>
       <geometry>
-        <box size="${robot_width} ${robot_height} ${robot_depth}"/>
-        <!-- <mesh filename="package://ros_gazebo/meshes/AMR_250.stl" scale="0.001 0.001 0.001"/> -->
+        <!-- <box size="${robot_width} ${robot_height} ${robot_depth}"/> -->
+        <mesh filename="package://ros_gazebo/meshes/AMR_250.stl" scale="0.001 0.001 0.001"/>
       </geometry>
+      <surface>
+        <friction>
+          <ode>
+            <mu>0</mu>
+            <mu2>0</mu2>
+            <slip1>1.0</slip1>
+            <slip2>1.0</slip2>
+          </ode>
+        </friction>
+      </surface>
     </collision>
   </link>
@@ -63,5 +75,5 @@
       <material name="orange"/>
     </visual>
-    <collision>
+    <collision name="base_module_under">
       <origin xyz="0 0 0" rpy="0 0 0"/>
       <geometry>
@@ -88,5 +100,5 @@
       <material name="brown"/>
     </visual>
-    <collision>
+    <collision name="base_module_up">
       <origin xyz="0 0 0" rpy="0 0 0"/>
       <geometry>
@@ -119,5 +131,5 @@
       <material name="blue"/>
     </visual>
-    <collision>
+    <collision name="base_laser_front">
       <origin xyz="0 0 0" rpy="0 0 0"/>
       <geometry>
@@ -144,5 +156,5 @@
       <material name="blue"/>
     </visual>
-    <collision>
+    <collision name="base_laser_back">
       <origin xyz="0 0 0" rpy="0 0 0"/>
       <geometry>

Commit message: test good

File: ros_gazebo/urdf/robot.xacro (robot description, xacro)
@@ -15,18 +15,14 @@
 	<xacro:property name="module_width" value="0.664" />
   <xacro:property name="module_depth" value="0.15" />
-  <link name="base_footprint">
-    <origin xyz="0 0 0" rpy="0 0 -1.57"/>
-  </link>
+  <link name="base_footprint"></link>
   <link name="base_link">
-    <pose>0 0 0 0 0 0</pose>
     <inertial>
-      <origin xyz="0 0 -0.069" rpy="0 0 0"/>
+      <origin xyz="0 0 -0.068" rpy="0 0 0"/>
       <mass value="${robot_mass}" />
       <solid_cuboid_inertia m="${robot_mass}" h="${robot_height}" w="${robot_width}" d="${robot_depth}"/>
     </inertial>
     <visual>
-      <origin xyz="0 0 -0.069" rpy="0 0 0"/>
+      <origin xyz="0 0 -0.068" rpy="0 0 0"/>
       <geometry>
-        <!-- <box size="${robot_width} ${robot_height} ${robot_depth}"/> -->
         <mesh filename="package://ros_gazebo/meshes/AMR_250.stl" scale="0.001 0.001 0.001"/>
       </geometry>
@@ -34,7 +30,6 @@
     </visual>
     <collision name="base_link">
-      <origin xyz="0 0 -0.069" rpy="0 0 0"/>
+      <origin xyz="0 0 -0.068" rpy="0 0 0"/>
       <geometry>
-        <!-- <box size="${robot_width} ${robot_height} ${robot_depth}"/> -->
         <mesh filename="package://ros_gazebo/meshes/AMR_250.stl" scale="0.001 0.001 0.001"/>
       </geometry>
@@ -168,4 +163,29 @@
     <origin xyz="-0.483 -0.265 0" rpy="3.14 0 3.925"/>
   </joint>
+  <!-- <link name="base_trolley">
+    <inertial>
+      <origin xyz="0 0 0" rpy="0 0 0" />
+      <mass value="1" />
+      <solid_cuboid_inertia m="${module_mass}" h="${module_height}" w="${module_width}" d="${module_depth}"/>
+    </inertial>
+    <visual>
+      <origin xyz="0 0 0" rpy="0 0 0"/>
+      <geometry>
+        <mesh filename="package://ros_gazebo/meshes/AMR_Trolley.stl" scale="0.001 0.001 0.001"/>
+      </geometry>
+      <material name="blue"/>
+    </visual>
+    <collision name="base_trolley">
+      <origin xyz="0 0 0" rpy="0 0 0"/>
+      <geometry>
+        <mesh filename="package://ros_gazebo/meshes/AMR_Trolley.stl" scale="0.001 0.001 0.001"/>
+      </geometry>
+    </collision>
+  </link>
+  <joint name="base_trolley_joint" type="fixed">
+    <parent link="base_module_up"/>
+    <child link="base_trolley"/>
+    <origin xyz="-0 0 0" rpy="0 0 0"/>
+  </joint> -->
   <xacro:link_wheel name="right_wheel" />
   <xacro:joint_wheel name="joint_right_wheel" child="right_wheel" origin_xyz="0 -0.242 0" />

Commit message: save

File: ros_gazebo/urdf/robot.xacro (robot description, xacro)
@@ -163,29 +163,4 @@
     <origin xyz="-0.483 -0.265 0" rpy="3.14 0 3.925"/>
   </joint>
-  <!-- <link name="base_trolley">
-    <inertial>
-      <origin xyz="0 0 0" rpy="0 0 0" />
-      <mass value="1" />
-      <solid_cuboid_inertia m="${module_mass}" h="${module_height}" w="${module_width}" d="${module_depth}"/>
-    </inertial>
-    <visual>
-      <origin xyz="0 0 0" rpy="0 0 0"/>
-      <geometry>
-        <mesh filename="package://ros_gazebo/meshes/AMR_Trolley.stl" scale="0.001 0.001 0.001"/>
-      </geometry>
-      <material name="blue"/>
-    </visual>
-    <collision name="base_trolley">
-      <origin xyz="0 0 0" rpy="0 0 0"/>
-      <geometry>
-        <mesh filename="package://ros_gazebo/meshes/AMR_Trolley.stl" scale="0.001 0.001 0.001"/>
-      </geometry>
-    </collision>
-  </link>
-  <joint name="base_trolley_joint" type="fixed">
-    <parent link="base_module_up"/>
-    <child link="base_trolley"/>
-    <origin xyz="-0 0 0" rpy="0 0 0"/>
-  </joint> -->
   <xacro:link_wheel name="right_wheel" />
   <xacro:joint_wheel name="joint_right_wheel" child="right_wheel" origin_xyz="0 -0.242 0" />

Commit message: save

File: ros_gazebo/urdf/robot.xacro (robot description, xacro)
@@ -7,9 +7,9 @@
   <xacro:include filename="$(find ros_gazebo)/urdf/robot.gazebo" />
   <xacro:include filename="$(find ros_gazebo)/urdf/macros.xacro" />
-	<xacro:property name="robot_mass" value="5" />
+	<xacro:property name="robot_mass" value="3" />
 	<xacro:property name="robot_height" value="1.165" />
 	<xacro:property name="robot_width" value="0.664" />
   <xacro:property name="robot_depth" value="0.33" />
-	<xacro:property name="module_mass" value="5" />
+	<xacro:property name="module_mass" value="1" />
 	<xacro:property name="module_height" value="1.161" />
 	<xacro:property name="module_width" value="0.664" />
@@ -51,5 +51,5 @@
     <origin xyz="0.0 0.0 0.1" rpy="0 0 0"/>
   </joint>
-  <!-- <link name="base_module"></link>
+  <link name="base_module"></link>
   <joint name="base_module_joint" type="fixed">
     <parent link="base_link"/>
@@ -106,5 +106,5 @@
     <child link="base_module_up"/>
     <origin xyz="0.0 0.0 0.0" rpy="0 0 0"/>
-  </joint> -->
+  </joint>
   <link name="base_laser"></link>
   <joint name="base_laser_joint" type="fixed">

Commit message: save

File: ros_gazebo/urdf/robot.xacro (robot description, xacro)
@@ -7,9 +7,9 @@
   <xacro:include filename="$(find ros_gazebo)/urdf/robot.gazebo" />
   <xacro:include filename="$(find ros_gazebo)/urdf/macros.xacro" />
-	<xacro:property name="robot_mass" value="4" />
+	<xacro:property name="robot_mass" value="3" />
 	<xacro:property name="robot_height" value="1.165" />
 	<xacro:property name="robot_width" value="0.664" />
   <xacro:property name="robot_depth" value="0.33" />
-	<xacro:property name="module_mass" value="2" />
+	<xacro:property name="module_mass" value="1" />
 	<xacro:property name="module_height" value="1.161" />
 	<xacro:property name="module_width" value="0.664" />
@@ -18,10 +18,10 @@
   <link name="base_link">
     <inertial>
-      <origin xyz="0 0 -0.068" rpy="0 0 0"/>
+      <origin xyz="0 0 -0.069" rpy="0 0 0"/>
       <mass value="${robot_mass}" />
       <solid_cuboid_inertia m="${robot_mass}" h="${robot_height}" w="${robot_width}" d="${robot_depth}"/>
     </inertial>
     <visual>
-      <origin xyz="0 0 -0.068" rpy="0 0 0"/>
+      <origin xyz="0 0 -0.069" rpy="0 0 0"/>
       <geometry>
         <mesh filename="package://ros_gazebo/meshes/AMR_250.stl" scale="0.001 0.001 0.001"/>
@@ -30,5 +30,5 @@
     </visual>
     <collision name="base_link">
-      <origin xyz="0 0 -0.068" rpy="0 0 0"/>
+      <origin xyz="0 0 -0.069" rpy="0 0 0"/>
       <geometry>
         <mesh filename="package://ros_gazebo/meshes/AMR_250.stl" scale="0.001 0.001 0.001"/>

Commit message: save

File: ros_gazebo/urdf/robot.xacro (robot description, xacro)
@@ -163,4 +163,29 @@
     <origin xyz="-0.483 -0.265 0" rpy="3.14 0 3.925"/>
   </joint>
+  <link name="base_camera">
+    <inertial>
+      <origin xyz="0 0 0" rpy="0 0 0" />
+      <mass value="1" />
+      <xacro:cylinder_inertia mass="0.1" r="0.05" l="0.1" />
+    </inertial>
+    <visual>
+      <origin xyz="0 0 0" rpy="0 0 0"/>
+      <geometry>
+        <box size="0.02 0.1 0.02"/>
+      </geometry>
+      <material name="green"/>
+    </visual>
+    <collision name="base_laser_back">
+      <origin xyz="0 0 0" rpy="0 0 0"/>
+      <geometry>
+        <box size="0.02 0.1 0.02"/>
+      </geometry>
+    </collision>
+  </link>
+  <joint name="base_camera_joint" type="fixed">
+    <parent link="base_link"/>
+    <child link="base_camera"/>
+    <origin xyz="0.53 0 0.15" rpy="0 0 0"/>
+  </joint>
   <xacro:link_wheel name="right_wheel" />
   <xacro:joint_wheel name="joint_right_wheel" child="right_wheel" origin_xyz="0 -0.242 0" />

Commit message: save

File: ros_gazebo/urdf/robot.xacro (robot description, xacro)
@@ -7,5 +7,5 @@
   <xacro:include filename="$(find ros_gazebo)/urdf/robot.gazebo" />
   <xacro:include filename="$(find ros_gazebo)/urdf/macros.xacro" />
-	<xacro:property name="robot_mass" value="3" />
+	<xacro:property name="robot_mass" value="5" />
 	<xacro:property name="robot_height" value="1.165" />
 	<xacro:property name="robot_width" value="0.664" />

Commit message: update

File: ros_gazebo/urdf/robot.xacro (robot description, xacro)
@@ -51,5 +51,5 @@
     <origin xyz="0.0 0.0 0.1" rpy="0 0 0"/>
   </joint>
-  <link name="base_module"></link>
+  <!-- <link name="base_module"></link>
   <joint name="base_module_joint" type="fixed">
     <parent link="base_link"/>
@@ -106,6 +106,7 @@
     <child link="base_module_up"/>
     <origin xyz="0.0 0.0 0.0" rpy="0 0 0"/>
-  </joint>
-  <link name="base_laser"></link>
+  </joint> -->
+  <plugin name="LiftModuleWorld" filename="libLiftModuleWorld.so"/>
+  <!-- <link name="base_laser"></link>
   <joint name="base_laser_joint" type="fixed">
     <parent link="base_link"/>
@@ -187,5 +188,5 @@
     <child link="base_camera"/>
     <origin xyz="0.53 0 0.15" rpy="0 0 0"/>
-  </joint>
+  </joint> -->
   <xacro:link_wheel name="right_wheel" />
   <xacro:joint_wheel name="joint_right_wheel" child="right_wheel" origin_xyz="0 -0.242 0" />

Commit message: save

File: ros_gazebo/urdf/robot.xacro (robot description, xacro)
@@ -7,5 +7,5 @@
   <xacro:include filename="$(find ros_gazebo)/urdf/robot.gazebo" />
   <xacro:include filename="$(find ros_gazebo)/urdf/macros.xacro" />
-	<xacro:property name="robot_mass" value="5" />
+	<xacro:property name="robot_mass" value="2" />
 	<xacro:property name="robot_height" value="1.165" />
 	<xacro:property name="robot_width" value="0.664" />
